Commit message: Restructure experiment 3 as guided sensor installation

File: urdf/differential_robot.urdf.xacro (robot description, xacro)
@@ -1,295 +1,10 @@
 <?xml version="1.0"?>
 <robot xmlns:xacro="http://www.ros.org/wiki/xacro" name="gazebo_diffbot">
-  <xacro:arg name="enable_camera" default="true"/>
-  <xacro:arg name="enable_lidar" default="true"/>
-  <xacro:property name="base_length" value="0.60"/>
-  <xacro:property name="base_width" value="0.45"/>
-  <xacro:property name="base_height" value="0.20"/>
-  <xacro:property name="wheel_radius" value="0.10"/>
-  <xacro:property name="wheel_width" value="0.06"/>
-  <xacro:property name="wheel_separation" value="0.48"/>
-  <xacro:property name="sensor_mount_height" value="0.42"/>
-  <material name="blue">
-    <color rgba="0.08 0.25 0.65 1.0"/>
-  </material>
-  <material name="black">
-    <color rgba="0.03 0.03 0.03 1.0"/>
-  </material>
-  <material name="gray">
-    <color rgba="0.45 0.45 0.45 1.0"/>
-  </material>
-  <link name="base_link">
-    <visual>
-      <origin xyz="0 0 ${wheel_radius + base_height / 2}"/>
-      <geometry><box size="${base_length} ${base_width} ${base_height}"/></geometry>
-      <material name="blue"/>
-    </visual>
-    <collision>
-      <origin xyz="0 0 ${wheel_radius + base_height / 2}"/>
-      <geometry><box size="${base_length} ${base_width} ${base_height}"/></geometry>
-    </collision>
-    <inertial>
-      <origin xyz="0 0 ${wheel_radius + base_height / 2}"/>
-      <mass value="12.0"/>
-      <inertia ixx="0.25" ixy="0" ixz="0" iyy="0.40" iyz="0" izz="0.55"/>
-    </inertial>
-  </link>
-  <!-- Gazebo approximation of the Unitree Mid-360 mounting point. -->
-  <link name="mid360_link">
-    <visual>
-      <origin xyz="0 0 0"/>
-      <geometry><cylinder radius="0.045" length="0.07"/></geometry>
-      <material name="gray"/>
-    </visual>
-    <collision>
-      <origin xyz="0 0 0"/>
-      <geometry><cylinder radius="0.045" length="0.07"/></geometry>
-    </collision>
-    <inertial>
-      <mass value="0.25"/>
-      <inertia ixx="0.0001" ixy="0" ixz="0" iyy="0.0001" iyz="0" izz="0.0001"/>
-    </inertial>
-  </link>
-  <joint name="mid360_joint" type="fixed">
-    <parent link="base_link"/>
-    <child link="mid360_link"/>
-    <origin xyz="0 0 ${sensor_mount_height}"/>
-  </joint>
-  <!-- RGB camera frame used by the later YOLO pipeline. -->
-  <xacro:if value="$(arg enable_camera)">
-  <link name="camera_link">
-    <visual>
-      <origin xyz="0 0 0"/>
-      <geometry><box size="0.06 0.04 0.03"/></geometry>
-      <material name="black"/>
-    </visual>
-  </link>
-  <joint name="camera_joint" type="fixed">
-    <parent link="base_link"/>
-    <child link="camera_link"/>
-    <origin xyz="0.22 0 ${sensor_mount_height - 0.04}" rpy="0 0 0"/>
-  </joint>
-  </xacro:if>
-  <xacro:macro name="wheel" params="name y">
-    <link name="${name}_wheel_link">
-      <visual>
-        <origin rpy="1.57079632679 0 0"/>
-        <geometry><cylinder radius="${wheel_radius}" length="${wheel_width}"/></geometry>
-        <material name="black"/>
-      </visual>
-      <collision>
-        <origin rpy="1.57079632679 0 0"/>
-        <geometry><cylinder radius="${wheel_radius}" length="${wheel_width}"/></geometry>
-      </collision>
-      <inertial>
-        <mass value="1.0"/>
-        <inertia ixx="0.005" ixy="0" ixz="0" iyy="0.005" iyz="0" izz="0.005"/>
-      </inertial>
-    </link>
-    <joint name="${name}_wheel_joint" type="continuous">
-      <parent link="base_link"/>
-      <child link="${name}_wheel_link"/>
-      <origin xyz="0 ${y} ${wheel_radius}"/>
-      <axis xyz="0 1 0"/>
-    </joint>
-  </xacro:macro>
-  <xacro:wheel name="left" y="${wheel_separation / 2}"/>
-  <xacro:wheel name="right" y="-${wheel_separation / 2}"/>
-  <link name="caster_link">
-    <visual>
-      <origin xyz="0 0 ${wheel_radius}"/>
-      <geometry><sphere radius="0.06"/></geometry>
-      <material name="gray"/>
-    </visual>
-    <collision>
-      <origin xyz="0 0 ${wheel_radius}"/>
-      <geometry><sphere radius="0.06"/></geometry>
-    </collision>
-    <inertial>
-      <mass value="0.3"/>
-      <inertia ixx="0.0004" ixy="0" ixz="0" iyy="0.0004" iyz="0" izz="0.0004"/>
-    </inertial>
-  </link>
-  <joint name="caster_joint" type="fixed">
-    <parent link="base_link"/>
-    <child link="caster_link"/>
-    <origin xyz="-${base_length / 2 - 0.08} 0 0"/>
-  </joint>
-  <gazebo reference="base_link">
-    <material>Gazebo/Blue</material>
-  </gazebo>
-  <gazebo reference="left_wheel_link"><material>Gazebo/Black</material></gazebo>
-  <gazebo reference="right_wheel_link"><material>Gazebo/Black</material></gazebo>
-  <xacro:if value="$(arg enable_lidar)">
-  <gazebo reference="mid360_link">
-    <sensor name="mid360_lidar" type="ray">
-      <always_on>true</always_on>
-      <visualize>false</visualize>
-      <update_rate>10.0</update_rate>
-      <ray>
-        <scan>
-          <horizontal>
-            <samples>720</samples>
-            <resolution>1.0</resolution>
-            <min_angle>-3.14159265359</min_angle>
-            <max_angle>3.14159265359</max_angle>
-          </horizontal>
-          <vertical>
-            <samples>32</samples>
-            <resolution>1.0</resolution>
-            <min_angle>-0.5235987756</min_angle>
-            <max_angle>0.2617993878</max_angle>
-          </vertical>
-        </scan>
-        <range>
-          <min>0.10</min>
-          <max>70.0</max>
-          <resolution>0.01</resolution>
-        </range>
-      </ray>
-      <plugin name="mid360_pointcloud" filename="libgazebo_ros_ray_sensor.so">
-        <ros>
-          <namespace>/</namespace>
-          <remapping>~/out:=mid360/points</remapping>
-        </ros>
-        <output_type>sensor_msgs/PointCloud2</output_type>
-      </plugin>
-    </sensor>
-  </gazebo>
-  </xacro:if>
-  <xacro:if value="$(arg enable_camera)">
-  <gazebo reference="camera_link">
-    <sensor name="depth_camera" type="camera">
-      <always_on>true</always_on>
-      <visualize>false</visualize>
-      <update_rate>10.0</update_rate>
-      <camera name="depth_camera_optical">
-        <horizontal_fov>1.0472</horizontal_fov>
-        <image>
-          <width>320</width>
-          <height>240</height>
-          <format>R8G8B8</format>
-        </image>
-        <clip>
-          <near>0.05</near>
-          <far>20.0</far>
-        </clip>
-      </camera>
-      <plugin name="depth_camera_ros" filename="libgazebo_ros_camera.so">
-        <ros>
-          <namespace>/camera</namespace>
-          <remapping>image_raw:=color/image_raw</remapping>
-          <remapping>camera_info:=color/camera_info</remapping>
-        </ros>
-        <camera_name>depth_camera</camera_name>
-        <frame_name>camera_link</frame_name>
-      </plugin>
-    </sensor>
-  </gazebo>
-  </xacro:if>
-  <gazebo>
-    <plugin name="diff_drive" filename="libgazebo_ros_diff_drive.so">
-      <ros>
-        <namespace>/</namespace>
-      </ros>
-      <update_rate>50</update_rate>
-      <left_joint>left_wheel_joint</left_joint>
-      <right_joint>right_wheel_joint</right_joint>
-      <wheel_separation>${wheel_separation}</wheel_separation>
-      <wheel_diameter>${2 * wheel_radius}</wheel_diameter>
-      <max_wheel_torque>20</max_wheel_torque>
-      <max_wheel_acceleration>10</max_wheel_acceleration>
-      <command_topic>cmd_vel</command_topic>
-      <odometry_topic>odom</odometry_topic>
-      <odometry_frame>odom</odometry_frame>
-      <robot_base_frame>base_link</robot_base_frame>
-      <publish_odom>true</publish_odom>
-      <publish_odom_tf>true</publish_odom_tf>
-      <publish_wheel_tf>false</publish_wheel_tf>
-      <publish_wheel_joint_state>true</publish_wheel_joint_state>
-    </plugin>
-  </gazebo>
-    <link name="imu_link">
-    <visual>
-      <origin xyz="0 0 0"/>
-      <geometry>
-        <box size="0.06 0.04 0.02"/>
-      </geometry>
-      <material name="black"/>
-    </visual>
-    <collision>
-      <origin xyz="0 0 0"/>
-      <geometry>
-        <box size="0.06 0.04 0.02"/>
-      </geometry>
-    </collision>
-    <inertial>
-      <origin xyz="0 0 0"/>
-      <mass value="0.1"/>
-      <inertia ixx="0.0001" ixy="0" ixz="0"
-               iyy="0.0001" iyz="0" izz="0.0001"/>
-    </inertial>
-  </link>
-  <joint name="imu_joint" type="fixed">
-    <parent link="base_link"/>
-    <child link="imu_link"/>
-    <origin xyz="-0.15 0 ${sensor_mount_height - 0.08}" rpy="0 0 0"/>
-  </joint>
-  <gazebo reference="imu_link">
-    <sensor name="imu_sensor" type="imu">
-      <always_on>true</always_on>
-      <visualize>false</visualize>
-      <update_rate>100.0</update_rate>
-      <imu>
-        <angular_velocity>
-          <x>
-            <noise type="gaussian">
-              <mean>0.0</mean>
-              <stddev>0.001</stddev>
-            </noise>
-          </x>
-          <y>
-            <noise type="gaussian">
-              <mean>0.0</mean>
-              <stddev>0.001</stddev>
-            </noise>
-          </y>
-          <z>
-            <noise type="gaussian">
-              <mean>0.0</mean>
-              <stddev>0.001</stddev>
-            </noise>
-          </z>
-        </angular_velocity>
-        <linear_acceleration>
-          <x>
-            <noise type="gaussian">
-              <mean>0.0</mean>
-              <stddev>0.01</stddev>
-            </noise>
-          </x>
-          <y>
-            <noise type="gaussian">
-              <mean>0.0</mean>
-              <stddev>0.01</stddev>
-            </noise>
-          </y>
-          <z>
-            <noise type="gaussian">
-              <mean>0.0</mean>
-              <stddev>0.01</stddev>
-            </noise>
-          </z>
-        </linear_acceleration>
-      </imu>
-      <plugin name="imu_plugin"
-              filename="libgazebo_ros_imu_sensor.so">
-        <ros>
-          <namespace>/</namespace>
-          <remapping>~/out:=imu/data</remapping>
-        </ros>
-        <frame_name>imu_link</frame_name>
-      </plugin>
-    </sensor>
-  </gazebo>
+  <xacro:include filename="robot_base_macro.xacro"/>
+  <xacro:include filename="sensor_macros.xacro"/>
+  <!-- The mobile base is ready. Install the three sensors during Experiment 3. -->
+  <xacro:differential_robot_base/>
+  <!-- STEP 1: Install the camera below this line. -->
+  <!-- STEP 2: Install the Mid-360-like lidar below this line. -->
+  <!-- STEP 3: Install the IMU below this line. -->
 </robot>
