Commit message: Improve robot and sensor visual models

File: urdf/robot_base_macro.xacro (robot description, xacro)
@@ -1,23 +1,24 @@
 <?xml version="1.0"?>
 <robot xmlns:xacro="http://www.ros.org/wiki/xacro">
-  <xacro:macro name="differential_wheel" params="name y radius width">
+  <xacro:macro name="differential_wheel" params="name y radius width side">
     <link name="${name}_wheel_link">
-      <visual>
+      <visual name="tire">
         <origin rpy="1.57079632679 0 0"/>
-        <geometry>
-          <cylinder radius="${radius}" length="${width}"/>
-        </geometry>
-        <material name="black"/>
+        <geometry><cylinder radius="${radius}" length="${width}"/></geometry>
+        <material name="tire_black"/>
+      </visual>
+      <visual name="outer_hub">
+        <origin xyz="0 ${side * (width / 2 + 0.009)} 0" rpy="1.57079632679 0 0"/>
+        <geometry><cylinder radius="${radius * 0.48}" length="0.018"/></geometry>
+        <material name="hub_silver"/>
       </visual>
       <collision>
         <origin rpy="1.57079632679 0 0"/>
-        <geometry>
-          <cylinder radius="${radius}" length="${width}"/>
-        </geometry>
+        <geometry><cylinder radius="${radius}" length="${width}"/></geometry>
       </collision>
       <inertial>
-        <mass value="1.0"/>
-        <inertia ixx="0.005" ixy="0" ixz="0"
-                 iyy="0.005" iyz="0" izz="0.005"/>
+        <mass value="2.0"/>
+        <inertia ixx="0.018" ixy="0" ixz="0"
+                 iyy="0.018" iyz="0" izz="0.018"/>
       </inertial>
     </link>
@@ -30,68 +31,103 @@
   </xacro:macro>
   <xacro:macro name="differential_robot_base" params="">
-    <xacro:property name="base_length" value="0.60"/>
-    <xacro:property name="base_width" value="0.45"/>
-    <xacro:property name="base_height" value="0.20"/>
-    <xacro:property name="wheel_radius" value="0.10"/>
-    <xacro:property name="wheel_width" value="0.06"/>
-    <xacro:property name="wheel_separation" value="0.48"/>
-    <material name="blue">
-      <color rgba="0.08 0.25 0.65 1.0"/>
-    </material>
-    <material name="black">
-      <color rgba="0.03 0.03 0.03 1.0"/>
-    </material>
-    <material name="gray">
-      <color rgba="0.45 0.45 0.45 1.0"/>
-    </material>
+    <xacro:property name="base_length" value="1.10"/>
+    <xacro:property name="base_width" value="0.72"/>
+    <xacro:property name="base_height" value="0.24"/>
+    <xacro:property name="wheel_radius" value="0.18"/>
+    <xacro:property name="wheel_width" value="0.12"/>
+    <xacro:property name="wheel_separation" value="0.82"/>
+    <material name="body_blue"><color rgba="0.04 0.22 0.62 1"/></material>
+    <material name="body_dark"><color rgba="0.025 0.055 0.10 1"/></material>
+    <material name="deck_gray"><color rgba="0.32 0.38 0.44 1"/></material>
+    <material name="tire_black"><color rgba="0.015 0.015 0.02 1"/></material>
+    <material name="hub_silver"><color rgba="0.72 0.76 0.80 1"/></material>
+    <material name="sensor_black"><color rgba="0.025 0.03 0.035 1"/></material>
+    <material name="lens_blue"><color rgba="0.03 0.35 0.68 1"/></material>
+    <material name="light_white"><color rgba="1.0 0.92 0.60 1"/></material>
+    <material name="light_red"><color rgba="0.75 0.02 0.02 1"/></material>
+    <material name="axis_red"><color rgba="0.90 0.05 0.05 1"/></material>
     <link name="base_link">
-      <visual>
-        <origin xyz="0 0 ${wheel_radius + base_height / 2}"/>
-        <geometry>
-          <box size="${base_length} ${base_width} ${base_height}"/>
-        </geometry>
-        <material name="blue"/>
+      <visual name="lower_chassis">
+        <origin xyz="0 0 0.27"/>
+        <geometry><box size="${base_length} ${base_width} ${base_height}"/></geometry>
+        <material name="body_blue"/>
+      </visual>
+      <visual name="upper_body">
+        <origin xyz="-0.06 0 0.43"/>
+        <geometry><box size="0.78 0.58 0.12"/></geometry>
+        <material name="body_dark"/>
+      </visual>
+      <visual name="sensor_deck">
+        <origin xyz="0.02 0 0.515"/>
+        <geometry><box size="0.64 0.48 0.05"/></geometry>
+        <material name="deck_gray"/>
+      </visual>
+      <visual name="front_bumper">
+        <origin xyz="0.575 0 0.23"/>
+        <geometry><box size="0.05 0.76 0.16"/></geometry>
+        <material name="body_dark"/>
+      </visual>
+      <visual name="rear_bumper">
+        <origin xyz="-0.575 0 0.23"/>
+        <geometry><box size="0.05 0.76 0.16"/></geometry>
+        <material name="body_dark"/>
+      </visual>
+      <visual name="left_headlight">
+        <origin xyz="0.606 0.22 0.30" rpy="0 1.57079632679 0"/>
+        <geometry><cylinder radius="0.045" length="0.018"/></geometry>
+        <material name="light_white"/>
+      </visual>
+      <visual name="right_headlight">
+        <origin xyz="0.606 -0.22 0.30" rpy="0 1.57079632679 0"/>
+        <geometry><cylinder radius="0.045" length="0.018"/></geometry>
+        <material name="light_white"/>
+      </visual>
+      <visual name="left_taillight">
+        <origin xyz="-0.606 0.22 0.30" rpy="0 1.57079632679 0"/>
+        <geometry><cylinder radius="0.035" length="0.018"/></geometry>
+        <material name="light_red"/>
+      </visual>
+      <visual name="right_taillight">
+        <origin xyz="-0.606 -0.22 0.30" rpy="0 1.57079632679 0"/>
+        <geometry><cylinder radius="0.035" length="0.018"/></geometry>
+        <material name="light_red"/>
       </visual>
       <collision>
-        <origin xyz="0 0 ${wheel_radius + base_height / 2}"/>
-        <geometry>
-          <box size="${base_length} ${base_width} ${base_height}"/>
-        </geometry>
+        <origin xyz="0 0 0.27"/>
+        <geometry><box size="${base_length} ${base_width} ${base_height}"/></geometry>
       </collision>
       <inertial>
-        <origin xyz="0 0 ${wheel_radius + base_height / 2}"/>
-        <mass value="12.0"/>
-        <inertia ixx="0.25" ixy="0" ixz="0"
-                 iyy="0.40" iyz="0" izz="0.55"/>
+        <origin xyz="0 0 0.27"/>
+        <mass value="28.0"/>
+        <inertia ixx="1.55" ixy="0" ixz="0"
+                 iyy="3.05" iyz="0" izz="4.20"/>
       </inertial>
     </link>
     <xacro:differential_wheel
-      name="left"
-      y="${wheel_separation / 2}"
-      radius="${wheel_radius}"
-      width="${wheel_width}"/>
+      name="left" y="${wheel_separation / 2}"
+      radius="${wheel_radius}" width="${wheel_width}" side="1"/>
     <xacro:differential_wheel
-      name="right"
-      y="-${wheel_separation / 2}"
-      radius="${wheel_radius}"
-      width="${wheel_width}"/>
+      name="right" y="-${wheel_separation / 2}"
+      radius="${wheel_radius}" width="${wheel_width}" side="-1"/>
     <link name="caster_link">
-      <visual>
-        <origin xyz="0 0 ${wheel_radius}"/>
-        <geometry>
-          <sphere radius="0.06"/>
-        </geometry>
-        <material name="gray"/>
+      <visual name="caster_fork">
+        <origin xyz="0 0 0.15"/>
+        <geometry><cylinder radius="0.055" length="0.10"/></geometry>
+        <material name="hub_silver"/>
+      </visual>
+      <visual name="caster_wheel">
+        <origin xyz="0 0 0.08" rpy="1.57079632679 0 0"/>
+        <geometry><cylinder radius="0.08" length="0.055"/></geometry>
+        <material name="tire_black"/>
       </visual>
       <collision>
-        <origin xyz="0 0 ${wheel_radius}"/>
-        <geometry>
-          <sphere radius="0.06"/>
-        </geometry>
+        <origin xyz="0 0 0.08"/>
+        <geometry><sphere radius="0.08"/></geometry>
       </collision>
       <inertial>
-        <mass value="0.3"/>
-        <inertia ixx="0.0004" ixy="0" ixz="0"
-                 iyy="0.0004" iyz="0" izz="0.0004"/>
+        <origin xyz="0 0 0.08"/>
+        <mass value="0.8"/>
+        <inertia ixx="0.003" ixy="0" ixz="0"
+                 iyy="0.003" iyz="0" izz="0.003"/>
       </inertial>
     </link>
@@ -99,20 +135,9 @@
       <parent link="base_link"/>
       <child link="caster_link"/>
-      <origin xyz="-${base_length / 2 - 0.08} 0 0"/>
+      <origin xyz="-0.43 0 0"/>
     </joint>
-    <gazebo reference="base_link">
-      <material>Gazebo/Blue</material>
-    </gazebo>
-    <gazebo reference="left_wheel_link">
-      <material>Gazebo/Black</material>
-    </gazebo>
-    <gazebo reference="right_wheel_link">
-      <material>Gazebo/Black</material>
-    </gazebo>
     <gazebo>
       <plugin name="diff_drive" filename="libgazebo_ros_diff_drive.so">
-        <ros>
-          <namespace>/</namespace>
-        </ros>
+        <ros><namespace>/</namespace></ros>
         <update_rate>50</update_rate>
         <left_joint>left_wheel_joint</left_joint>
@@ -120,6 +145,6 @@
         <wheel_separation>${wheel_separation}</wheel_separation>
         <wheel_diameter>${2 * wheel_radius}</wheel_diameter>
-        <max_wheel_torque>20</max_wheel_torque>
-        <max_wheel_acceleration>10</max_wheel_acceleration>
+        <max_wheel_torque>45</max_wheel_torque>
+        <max_wheel_acceleration>6</max_wheel_acceleration>
         <command_topic>cmd_vel</command_topic>
         <odometry_topic>odom</odometry_topic>

File: urdf/sensor_macros.xacro (robot description, xacro)
@@ -4,10 +4,25 @@
                params="parent frame optical_frame xyz rpy image_topic info_topic update_rate">
     <link name="${frame}">
-      <visual>
-        <geometry><box size="0.06 0.04 0.03"/></geometry>
-        <material name="black"/>
+      <visual name="camera_body">
+        <geometry><box size="0.14 0.10 0.08"/></geometry>
+        <material name="sensor_black"/>
+      </visual>
+      <visual name="camera_face">
+        <origin xyz="0.076 0 0"/>
+        <geometry><box size="0.015 0.09 0.07"/></geometry>
+        <material name="deck_gray"/>
+      </visual>
+      <visual name="camera_lens">
+        <origin xyz="0.095 0 0" rpy="0 1.57079632679 0"/>
+        <geometry><cylinder radius="0.032" length="0.04"/></geometry>
+        <material name="lens_blue"/>
+      </visual>
+      <visual name="camera_bracket">
+        <origin xyz="-0.035 0 -0.075"/>
+        <geometry><box size="0.035 0.08 0.08"/></geometry>
+        <material name="deck_gray"/>
       </visual>
       <collision>
-        <geometry><box size="0.06 0.04 0.03"/></geometry>
+        <geometry><box size="0.14 0.10 0.08"/></geometry>
       </collision>
       <inertial>
@@ -61,9 +76,23 @@
     <link name="${frame}">
       <visual>
-        <geometry><cylinder radius="0.045" length="0.07"/></geometry>
-        <material name="gray"/>
+        <geometry><cylinder radius="0.08" length="0.11"/></geometry>
+        <material name="sensor_black"/>
+      </visual>
+      <visual name="lidar_scan_band">
+        <geometry><cylinder radius="0.084" length="0.045"/></geometry>
+        <material name="lens_blue"/>
+      </visual>
+      <visual name="lidar_cap">
+        <origin xyz="0 0 0.065"/>
+        <geometry><cylinder radius="0.065" length="0.025"/></geometry>
+        <material name="deck_gray"/>
+      </visual>
+      <visual name="lidar_mount">
+        <origin xyz="0 0 -0.095"/>
+        <geometry><cylinder radius="0.045" length="0.08"/></geometry>
+        <material name="deck_gray"/>
       </visual>
       <collision>
-        <geometry><cylinder radius="0.045" length="0.07"/></geometry>
+        <geometry><cylinder radius="0.08" length="0.11"/></geometry>
       </collision>
       <inertial>
@@ -118,10 +147,20 @@
                params="parent frame xyz rpy topic update_rate">
     <link name="${frame}">
-      <visual>
-        <geometry><box size="0.06 0.04 0.02"/></geometry>
-        <material name="black"/>
+      <visual name="imu_body">
+        <geometry><box size="0.12 0.09 0.04"/></geometry>
+        <material name="sensor_black"/>
+      </visual>
+      <visual name="imu_top">
+        <origin xyz="0 0 0.023"/>
+        <geometry><box size="0.10 0.07 0.008"/></geometry>
+        <material name="deck_gray"/>
+      </visual>
+      <visual name="imu_forward_marker">
+        <origin xyz="0.045 0 0.031"/>
+        <geometry><box size="0.045 0.012 0.009"/></geometry>
+        <material name="axis_red"/>
       </visual>
       <collision>
-        <geometry><box size="0.06 0.04 0.02"/></geometry>
+        <geometry><box size="0.12 0.09 0.04"/></geometry>
       </collision>
       <inertial>

Commit message: Adjust wheel layout and Gazebo materials

File: urdf/robot_base_macro.xacro (robot description, xacro)
@@ -1,5 +1,5 @@
 <?xml version="1.0"?>
 <robot xmlns:xacro="http://www.ros.org/wiki/xacro">
-  <xacro:macro name="differential_wheel" params="name y radius width side">
+  <xacro:macro name="differential_wheel" params="name x y radius width side">
     <link name="${name}_wheel_link">
       <visual name="tire">
@@ -26,5 +26,5 @@
       <parent link="base_link"/>
       <child link="${name}_wheel_link"/>
-      <origin xyz="0 ${y} ${radius}"/>
+      <origin xyz="${x} ${y} ${radius}"/>
       <axis xyz="0 1 0"/>
     </joint>
@@ -105,29 +105,29 @@
     </link>
     <xacro:differential_wheel
-      name="left" y="${wheel_separation / 2}"
+      name="left" x="0.25" y="${wheel_separation / 2}"
       radius="${wheel_radius}" width="${wheel_width}" side="1"/>
     <xacro:differential_wheel
-      name="right" y="-${wheel_separation / 2}"
+      name="right" x="0.25" y="-${wheel_separation / 2}"
       radius="${wheel_radius}" width="${wheel_width}" side="-1"/>
     <link name="caster_link">
       <visual name="caster_fork">
-        <origin xyz="0 0 0.15"/>
-        <geometry><cylinder radius="0.055" length="0.10"/></geometry>
+        <origin xyz="0 0 0.225"/>
+        <geometry><cylinder radius="0.075" length="0.19"/></geometry>
         <material name="hub_silver"/>
       </visual>
       <visual name="caster_wheel">
-        <origin xyz="0 0 0.08" rpy="1.57079632679 0 0"/>
-        <geometry><cylinder radius="0.08" length="0.055"/></geometry>
+        <origin xyz="0 0 0.13" rpy="1.57079632679 0 0"/>
+        <geometry><cylinder radius="0.13" length="0.09"/></geometry>
         <material name="tire_black"/>
       </visual>
       <collision>
-        <origin xyz="0 0 0.08"/>
-        <geometry><sphere radius="0.08"/></geometry>
+        <origin xyz="0 0 0.13"/>
+        <geometry><sphere radius="0.13"/></geometry>
       </collision>
       <inertial>
-        <origin xyz="0 0 0.08"/>
-        <mass value="0.8"/>
-        <inertia ixx="0.003" ixy="0" ixz="0"
-                 iyy="0.003" iyz="0" izz="0.003"/>
+        <origin xyz="0 0 0.13"/>
+        <mass value="1.2"/>
+        <inertia ixx="0.008" ixy="0" ixz="0"
+                 iyy="0.008" iyz="0" izz="0.008"/>
       </inertial>
     </link>
@@ -137,4 +137,8 @@
       <origin xyz="-0.43 0 0"/>
     </joint>
+    <gazebo reference="base_link"><material>Gazebo/Blue</material></gazebo>
+    <gazebo reference="left_wheel_link"><material>Gazebo/Black</material></gazebo>
+    <gazebo reference="right_wheel_link"><material>Gazebo/Black</material></gazebo>
+    <gazebo reference="caster_link"><material>Gazebo/Black</material></gazebo>
     <gazebo>
       <plugin name="diff_drive" filename="libgazebo_ros_diff_drive.so">

File: urdf/sensor_macros.xacro (robot description, xacro)
@@ -44,4 +44,5 @@
     </joint>
     <gazebo reference="${frame}">
+      <material>Gazebo/Black</material>
       <sensor name="camera_sensor" type="camera">
         <always_on>true</always_on>
@@ -108,4 +109,5 @@
     </joint>
     <gazebo reference="${frame}">
+      <material>Gazebo/DarkGrey</material>
       <sensor name="mid360_lidar" type="ray">
         <always_on>true</always_on>
@@ -176,4 +178,5 @@
     </joint>
     <gazebo reference="${frame}">
+      <material>Gazebo/Grey</material>
       <sensor name="imu_sensor" type="imu">
         <always_on>true</always_on>
