Commit message: Embed colors in individual model visuals

File: urdf/robot_base_macro.xacro (robot description, xacro)
@@ -6,10 +6,10 @@
         <origin rpy="1.57079632679 0 0"/>
         <geometry><cylinder radius="${radius}" length="${width}"/></geometry>
-        <material name="tire_black"/>
+        <material name="${name}_tire_black"><color rgba="0.015 0.015 0.02 1"/></material>
       </visual>
       <visual name="outer_hub">
         <origin xyz="0 ${side * (width / 2 + 0.009)} 0" rpy="1.57079632679 0 0"/>
         <geometry><cylinder radius="${radius * 0.48}" length="0.018"/></geometry>
-        <material name="hub_silver"/>
+        <material name="${name}_hub_silver"><color rgba="0.72 0.76 0.80 1"/></material>
       </visual>
       <collision>
@@ -37,59 +37,49 @@
     <xacro:property name="wheel_width" value="0.12"/>
     <xacro:property name="wheel_separation" value="0.82"/>
-    <material name="body_blue"><color rgba="0.04 0.22 0.62 1"/></material>
-    <material name="body_dark"><color rgba="0.025 0.055 0.10 1"/></material>
-    <material name="deck_gray"><color rgba="0.32 0.38 0.44 1"/></material>
-    <material name="tire_black"><color rgba="0.015 0.015 0.02 1"/></material>
-    <material name="hub_silver"><color rgba="0.72 0.76 0.80 1"/></material>
-    <material name="sensor_black"><color rgba="0.025 0.03 0.035 1"/></material>
-    <material name="lens_blue"><color rgba="0.03 0.35 0.68 1"/></material>
-    <material name="light_white"><color rgba="1.0 0.92 0.60 1"/></material>
-    <material name="light_red"><color rgba="0.75 0.02 0.02 1"/></material>
-    <material name="axis_red"><color rgba="0.90 0.05 0.05 1"/></material>
     <link name="base_link">
       <visual name="lower_chassis">
         <origin xyz="0 0 0.27"/>
         <geometry><box size="${base_length} ${base_width} ${base_height}"/></geometry>
-        <material name="body_blue"/>
+        <material name="body_blue"><color rgba="0.04 0.22 0.62 1"/></material>
       </visual>
       <visual name="upper_body">
         <origin xyz="-0.06 0 0.43"/>
         <geometry><box size="0.78 0.58 0.12"/></geometry>
-        <material name="body_dark"/>
+        <material name="upper_body_dark"><color rgba="0.025 0.055 0.10 1"/></material>
       </visual>
       <visual name="sensor_deck">
         <origin xyz="0.02 0 0.515"/>
         <geometry><box size="0.64 0.48 0.05"/></geometry>
-        <material name="deck_gray"/>
+        <material name="deck_gray"><color rgba="0.32 0.38 0.44 1"/></material>
       </visual>
       <visual name="front_bumper">
         <origin xyz="0.575 0 0.23"/>
         <geometry><box size="0.05 0.76 0.16"/></geometry>
-        <material name="body_dark"/>
+        <material name="front_bumper_dark"><color rgba="0.025 0.055 0.10 1"/></material>
       </visual>
       <visual name="rear_bumper">
         <origin xyz="-0.575 0 0.23"/>
         <geometry><box size="0.05 0.76 0.16"/></geometry>
-        <material name="body_dark"/>
+        <material name="rear_bumper_dark"><color rgba="0.025 0.055 0.10 1"/></material>
       </visual>
       <visual name="left_headlight">
         <origin xyz="0.606 0.22 0.30" rpy="0 1.57079632679 0"/>
         <geometry><cylinder radius="0.045" length="0.018"/></geometry>
-        <material name="light_white"/>
+        <material name="left_headlight_white"><color rgba="1.0 0.92 0.60 1"/></material>
       </visual>
       <visual name="right_headlight">
         <origin xyz="0.606 -0.22 0.30" rpy="0 1.57079632679 0"/>
         <geometry><cylinder radius="0.045" length="0.018"/></geometry>
-        <material name="light_white"/>
+        <material name="right_headlight_white"><color rgba="1.0 0.92 0.60 1"/></material>
       </visual>
       <visual name="left_taillight">
         <origin xyz="-0.606 0.22 0.30" rpy="0 1.57079632679 0"/>
         <geometry><cylinder radius="0.035" length="0.018"/></geometry>
-        <material name="light_red"/>
+        <material name="left_taillight_red"><color rgba="0.75 0.02 0.02 1"/></material>
       </visual>
       <visual name="right_taillight">
         <origin xyz="-0.606 -0.22 0.30" rpy="0 1.57079632679 0"/>
         <geometry><cylinder radius="0.035" length="0.018"/></geometry>
-        <material name="light_red"/>
+        <material name="right_taillight_red"><color rgba="0.75 0.02 0.02 1"/></material>
       </visual>
       <collision>
@@ -114,10 +104,10 @@
         <origin xyz="0 0 0.225"/>
         <geometry><cylinder radius="0.075" length="0.19"/></geometry>
-        <material name="hub_silver"/>
+        <material name="caster_hub_silver"><color rgba="0.72 0.76 0.80 1"/></material>
       </visual>
       <visual name="caster_wheel">
         <origin xyz="0 0 0.13" rpy="1.57079632679 0 0"/>
         <geometry><cylinder radius="0.13" length="0.09"/></geometry>
-        <material name="tire_black"/>
+        <material name="caster_tire_black"><color rgba="0.015 0.015 0.02 1"/></material>
       </visual>
       <collision>
@@ -137,8 +127,4 @@
       <origin xyz="-0.43 0 0"/>
     </joint>
-    <gazebo reference="base_link"><material>Gazebo/Blue</material></gazebo>
-    <gazebo reference="left_wheel_link"><material>Gazebo/Black</material></gazebo>
-    <gazebo reference="right_wheel_link"><material>Gazebo/Black</material></gazebo>
-    <gazebo reference="caster_link"><material>Gazebo/Black</material></gazebo>
     <gazebo>
       <plugin name="diff_drive" filename="libgazebo_ros_diff_drive.so">

File: urdf/sensor_macros.xacro (robot description, xacro)
@@ -6,20 +6,20 @@
       <visual name="camera_body">
         <geometry><box size="0.14 0.10 0.08"/></geometry>
-        <material name="sensor_black"/>
+        <material name="camera_black"><color rgba="0.025 0.03 0.035 1"/></material>
       </visual>
       <visual name="camera_face">
         <origin xyz="0.076 0 0"/>
         <geometry><box size="0.015 0.09 0.07"/></geometry>
-        <material name="deck_gray"/>
+        <material name="camera_face_gray"><color rgba="0.32 0.38 0.44 1"/></material>
       </visual>
       <visual name="camera_lens">
         <origin xyz="0.095 0 0" rpy="0 1.57079632679 0"/>
         <geometry><cylinder radius="0.032" length="0.04"/></geometry>
-        <material name="lens_blue"/>
+        <material name="camera_lens_blue"><color rgba="0.03 0.35 0.68 1"/></material>
       </visual>
       <visual name="camera_bracket">
         <origin xyz="-0.035 0 -0.075"/>
         <geometry><box size="0.035 0.08 0.08"/></geometry>
-        <material name="deck_gray"/>
+        <material name="camera_bracket_gray"><color rgba="0.32 0.38 0.44 1"/></material>
       </visual>
       <collision>
@@ -44,5 +44,4 @@
     </joint>
     <gazebo reference="${frame}">
-      <material>Gazebo/Black</material>
       <sensor name="camera_sensor" type="camera">
         <always_on>true</always_on>
@@ -78,19 +77,19 @@
       <visual>
         <geometry><cylinder radius="0.08" length="0.11"/></geometry>
-        <material name="sensor_black"/>
+        <material name="lidar_black"><color rgba="0.025 0.03 0.035 1"/></material>
       </visual>
       <visual name="lidar_scan_band">
         <geometry><cylinder radius="0.084" length="0.045"/></geometry>
-        <material name="lens_blue"/>
+        <material name="lidar_band_blue"><color rgba="0.03 0.35 0.68 1"/></material>
       </visual>
       <visual name="lidar_cap">
         <origin xyz="0 0 0.065"/>
         <geometry><cylinder radius="0.065" length="0.025"/></geometry>
-        <material name="deck_gray"/>
+        <material name="lidar_cap_gray"><color rgba="0.32 0.38 0.44 1"/></material>
       </visual>
       <visual name="lidar_mount">
         <origin xyz="0 0 -0.095"/>
         <geometry><cylinder radius="0.045" length="0.08"/></geometry>
-        <material name="deck_gray"/>
+        <material name="lidar_mount_gray"><color rgba="0.32 0.38 0.44 1"/></material>
       </visual>
       <collision>
@@ -109,5 +108,4 @@
     </joint>
     <gazebo reference="${frame}">
-      <material>Gazebo/DarkGrey</material>
       <sensor name="mid360_lidar" type="ray">
         <always_on>true</always_on>
@@ -151,15 +149,15 @@
       <visual name="imu_body">
         <geometry><box size="0.12 0.09 0.04"/></geometry>
-        <material name="sensor_black"/>
+        <material name="imu_black"><color rgba="0.025 0.03 0.035 1"/></material>
       </visual>
       <visual name="imu_top">
         <origin xyz="0 0 0.023"/>
         <geometry><box size="0.10 0.07 0.008"/></geometry>
-        <material name="deck_gray"/>
+        <material name="imu_top_gray"><color rgba="0.32 0.38 0.44 1"/></material>
       </visual>
       <visual name="imu_forward_marker">
         <origin xyz="0.045 0 0.031"/>
         <geometry><box size="0.045 0.012 0.009"/></geometry>
-        <material name="axis_red"/>
+        <material name="imu_axis_red"><color rgba="0.90 0.05 0.05 1"/></material>
       </visual>
       <collision>
@@ -178,5 +176,4 @@
     </joint>
     <gazebo reference="${frame}">
-      <material>Gazebo/Grey</material>
       <sensor name="imu_sensor" type="imu">
         <always_on>true</always_on>

Commit message: Split visual parts for reliable Gazebo materials

File: urdf/robot_base_macro.xacro (robot description, xacro)
@@ -1,15 +1,40 @@
 <?xml version="1.0"?>
 <robot xmlns:xacro="http://www.ros.org/wiki/xacro">
+  <xacro:macro name="fixed_box_visual"
+               params="name parent xyz rpy size gazebo_material rgba">
+    <link name="${name}">
+      <visual>
+        <geometry><box size="${size}"/></geometry>
+        <material name="${name}_color"><color rgba="${rgba}"/></material>
+      </visual>
+    </link>
+    <joint name="${name}_joint" type="fixed">
+      <parent link="${parent}"/>
+      <child link="${name}"/>
+      <origin xyz="${xyz}" rpy="${rpy}"/>
+    </joint>
+    <gazebo reference="${name}"><material>${gazebo_material}</material></gazebo>
+  </xacro:macro>
+  <xacro:macro name="fixed_cylinder_visual"
+               params="name parent xyz rpy radius length gazebo_material rgba">
+    <link name="${name}">
+      <visual>
+        <geometry><cylinder radius="${radius}" length="${length}"/></geometry>
+        <material name="${name}_color"><color rgba="${rgba}"/></material>
+      </visual>
+    </link>
+    <joint name="${name}_joint" type="fixed">
+      <parent link="${parent}"/>
+      <child link="${name}"/>
+      <origin xyz="${xyz}" rpy="${rpy}"/>
+    </joint>
+    <gazebo reference="${name}"><material>${gazebo_material}</material></gazebo>
+  </xacro:macro>
   <xacro:macro name="differential_wheel" params="name x y radius width side">
     <link name="${name}_wheel_link">
-      <visual name="tire">
+      <visual>
         <origin rpy="1.57079632679 0 0"/>
         <geometry><cylinder radius="${radius}" length="${width}"/></geometry>
-        <material name="${name}_tire_black"><color rgba="0.015 0.015 0.02 1"/></material>
-      </visual>
-      <visual name="outer_hub">
-        <origin xyz="0 ${side * (width / 2 + 0.009)} 0" rpy="1.57079632679 0 0"/>
-        <geometry><cylinder radius="${radius * 0.48}" length="0.018"/></geometry>
-        <material name="${name}_hub_silver"><color rgba="0.72 0.76 0.80 1"/></material>
+        <material name="${name}_tire_color"><color rgba="0.015 0.015 0.02 1"/></material>
       </visual>
       <collision>
@@ -29,4 +54,11 @@
       <axis xyz="0 1 0"/>
     </joint>
+    <gazebo reference="${name}_wheel_link"><material>Gazebo/Black</material></gazebo>
+    <xacro:fixed_cylinder_visual
+      name="${name}_wheel_hub" parent="${name}_wheel_link"
+      xyz="0 ${side * (width / 2 + 0.009)} 0"
+      rpy="1.57079632679 0 0"
+      radius="${radius * 0.48}" length="0.018"
+      gazebo_material="Gazebo/Grey" rgba="0.72 0.76 0.80 1"/>
   </xacro:macro>
   <xacro:macro name="differential_robot_base" params="">
@@ -38,48 +70,8 @@
     <xacro:property name="wheel_separation" value="0.82"/>
     <link name="base_link">
-      <visual name="lower_chassis">
+      <visual>
         <origin xyz="0 0 0.27"/>
         <geometry><box size="${base_length} ${base_width} ${base_height}"/></geometry>
-        <material name="body_blue"><color rgba="0.04 0.22 0.62 1"/></material>
-      </visual>
-      <visual name="upper_body">
-        <origin xyz="-0.06 0 0.43"/>
-        <geometry><box size="0.78 0.58 0.12"/></geometry>
-        <material name="upper_body_dark"><color rgba="0.025 0.055 0.10 1"/></material>
-      </visual>
-      <visual name="sensor_deck">
-        <origin xyz="0.02 0 0.515"/>
-        <geometry><box size="0.64 0.48 0.05"/></geometry>
-        <material name="deck_gray"><color rgba="0.32 0.38 0.44 1"/></material>
-      </visual>
-      <visual name="front_bumper">
-        <origin xyz="0.575 0 0.23"/>
-        <geometry><box size="0.05 0.76 0.16"/></geometry>
-        <material name="front_bumper_dark"><color rgba="0.025 0.055 0.10 1"/></material>
-      </visual>
-      <visual name="rear_bumper">
-        <origin xyz="-0.575 0 0.23"/>
-        <geometry><box size="0.05 0.76 0.16"/></geometry>
-        <material name="rear_bumper_dark"><color rgba="0.025 0.055 0.10 1"/></material>
-      </visual>
-      <visual name="left_headlight">
-        <origin xyz="0.606 0.22 0.30" rpy="0 1.57079632679 0"/>
-        <geometry><cylinder radius="0.045" length="0.018"/></geometry>
-        <material name="left_headlight_white"><color rgba="1.0 0.92 0.60 1"/></material>
-      </visual>
-      <visual name="right_headlight">
-        <origin xyz="0.606 -0.22 0.30" rpy="0 1.57079632679 0"/>
-        <geometry><cylinder radius="0.045" length="0.018"/></geometry>
-        <material name="right_headlight_white"><color rgba="1.0 0.92 0.60 1"/></material>
-      </visual>
-      <visual name="left_taillight">
-        <origin xyz="-0.606 0.22 0.30" rpy="0 1.57079632679 0"/>
-        <geometry><cylinder radius="0.035" length="0.018"/></geometry>
-        <material name="left_taillight_red"><color rgba="0.75 0.02 0.02 1"/></material>
-      </visual>
-      <visual name="right_taillight">
-        <origin xyz="-0.606 -0.22 0.30" rpy="0 1.57079632679 0"/>
-        <geometry><cylinder radius="0.035" length="0.018"/></geometry>
-        <material name="right_taillight_red"><color rgba="0.75 0.02 0.02 1"/></material>
+        <material name="base_blue"><color rgba="0.04 0.22 0.62 1"/></material>
       </visual>
       <collision>
@@ -94,4 +86,41 @@
       </inertial>
     </link>
+    <gazebo reference="base_link"><material>Gazebo/Blue</material></gazebo>
+    <xacro:fixed_box_visual
+      name="upper_body_link" parent="base_link"
+      xyz="-0.06 0 0.43" rpy="0 0 0" size="0.78 0.58 0.12"
+      gazebo_material="Gazebo/Black" rgba="0.025 0.055 0.10 1"/>
+    <xacro:fixed_box_visual
+      name="sensor_deck_link" parent="base_link"
+      xyz="0.02 0 0.515" rpy="0 0 0" size="0.64 0.48 0.05"
+      gazebo_material="Gazebo/Grey" rgba="0.32 0.38 0.44 1"/>
+    <xacro:fixed_box_visual
+      name="front_bumper_link" parent="base_link"
+      xyz="0.575 0 0.23" rpy="0 0 0" size="0.05 0.76 0.16"
+      gazebo_material="Gazebo/Black" rgba="0.025 0.055 0.10 1"/>
+    <xacro:fixed_box_visual
+      name="rear_bumper_link" parent="base_link"
+      xyz="-0.575 0 0.23" rpy="0 0 0" size="0.05 0.76 0.16"
+      gazebo_material="Gazebo/Black" rgba="0.025 0.055 0.10 1"/>
+    <xacro:fixed_cylinder_visual
+      name="left_headlight_link" parent="base_link"
+      xyz="0.606 0.22 0.30" rpy="0 1.57079632679 0"
+      radius="0.045" length="0.018"
+      gazebo_material="Gazebo/Yellow" rgba="1.0 0.92 0.20 1"/>
+    <xacro:fixed_cylinder_visual
+      name="right_headlight_link" parent="base_link"
+      xyz="0.606 -0.22 0.30" rpy="0 1.57079632679 0"
+      radius="0.045" length="0.018"
+      gazebo_material="Gazebo/Yellow" rgba="1.0 0.92 0.20 1"/>
+    <xacro:fixed_cylinder_visual
+      name="left_taillight_link" parent="base_link"
+      xyz="-0.606 0.22 0.30" rpy="0 1.57079632679 0"
+      radius="0.035" length="0.018"
+      gazebo_material="Gazebo/Red" rgba="0.75 0.02 0.02 1"/>
+    <xacro:fixed_cylinder_visual
+      name="right_taillight_link" parent="base_link"
+      xyz="-0.606 -0.22 0.30" rpy="0 1.57079632679 0"
+      radius="0.035" length="0.018"
+      gazebo_material="Gazebo/Red" rgba="0.75 0.02 0.02 1"/>
     <xacro:differential_wheel
       name="left" x="0.25" y="${wheel_separation / 2}"
@@ -101,13 +130,8 @@
       radius="${wheel_radius}" width="${wheel_width}" side="-1"/>
     <link name="caster_link">
-      <visual name="caster_fork">
-        <origin xyz="0 0 0.225"/>
-        <geometry><cylinder radius="0.075" length="0.19"/></geometry>
-        <material name="caster_hub_silver"><color rgba="0.72 0.76 0.80 1"/></material>
-      </visual>
-      <visual name="caster_wheel">
+      <visual>
         <origin xyz="0 0 0.13" rpy="1.57079632679 0 0"/>
         <geometry><cylinder radius="0.13" length="0.09"/></geometry>
-        <material name="caster_tire_black"><color rgba="0.015 0.015 0.02 1"/></material>
+        <material name="caster_black"><color rgba="0.015 0.015 0.02 1"/></material>
       </visual>
       <collision>
@@ -127,4 +151,10 @@
       <origin xyz="-0.43 0 0"/>
     </joint>
+    <gazebo reference="caster_link"><material>Gazebo/Black</material></gazebo>
+    <xacro:fixed_cylinder_visual
+      name="caster_fork_link" parent="caster_link"
+      xyz="0 0 0.225" rpy="0 0 0"
+      radius="0.075" length="0.19"
+      gazebo_material="Gazebo/Grey" rgba="0.72 0.76 0.80 1"/>
     <gazebo>
       <plugin name="diff_drive" filename="libgazebo_ros_diff_drive.so">

File: urdf/sensor_macros.xacro (robot description, xacro)
@@ -4,22 +4,7 @@
                params="parent frame optical_frame xyz rpy image_topic info_topic update_rate">
     <link name="${frame}">
-      <visual name="camera_body">
+      <visual>
         <geometry><box size="0.14 0.10 0.08"/></geometry>
         <material name="camera_black"><color rgba="0.025 0.03 0.035 1"/></material>
-      </visual>
-      <visual name="camera_face">
-        <origin xyz="0.076 0 0"/>
-        <geometry><box size="0.015 0.09 0.07"/></geometry>
-        <material name="camera_face_gray"><color rgba="0.32 0.38 0.44 1"/></material>
-      </visual>
-      <visual name="camera_lens">
-        <origin xyz="0.095 0 0" rpy="0 1.57079632679 0"/>
-        <geometry><cylinder radius="0.032" length="0.04"/></geometry>
-        <material name="camera_lens_blue"><color rgba="0.03 0.35 0.68 1"/></material>
-      </visual>
-      <visual name="camera_bracket">
-        <origin xyz="-0.035 0 -0.075"/>
-        <geometry><box size="0.035 0.08 0.08"/></geometry>
-        <material name="camera_bracket_gray"><color rgba="0.32 0.38 0.44 1"/></material>
       </visual>
       <collision>
@@ -37,4 +22,18 @@
       <origin xyz="${xyz}" rpy="${rpy}"/>
     </joint>
+    <gazebo reference="${frame}"><material>Gazebo/Black</material></gazebo>
+    <xacro:fixed_box_visual
+      name="${frame}_face_link" parent="${frame}"
+      xyz="0.076 0 0" rpy="0 0 0" size="0.015 0.09 0.07"
+      gazebo_material="Gazebo/Grey" rgba="0.32 0.38 0.44 1"/>
+    <xacro:fixed_cylinder_visual
+      name="${frame}_lens_link" parent="${frame}"
+      xyz="0.095 0 0" rpy="0 1.57079632679 0"
+      radius="0.032" length="0.04"
+      gazebo_material="Gazebo/Blue" rgba="0.03 0.35 0.68 1"/>
+    <xacro:fixed_box_visual
+      name="${frame}_bracket_link" parent="${frame}"
+      xyz="-0.035 0 -0.075" rpy="0 0 0" size="0.035 0.08 0.08"
+      gazebo_material="Gazebo/Grey" rgba="0.32 0.38 0.44 1"/>
     <link name="${optical_frame}"/>
     <joint name="${optical_frame}_joint" type="fixed">
@@ -79,18 +78,4 @@
         <material name="lidar_black"><color rgba="0.025 0.03 0.035 1"/></material>
       </visual>
-      <visual name="lidar_scan_band">
-        <geometry><cylinder radius="0.084" length="0.045"/></geometry>
-        <material name="lidar_band_blue"><color rgba="0.03 0.35 0.68 1"/></material>
-      </visual>
-      <visual name="lidar_cap">
-        <origin xyz="0 0 0.065"/>
-        <geometry><cylinder radius="0.065" length="0.025"/></geometry>
-        <material name="lidar_cap_gray"><color rgba="0.32 0.38 0.44 1"/></material>
-      </visual>
-      <visual name="lidar_mount">
-        <origin xyz="0 0 -0.095"/>
-        <geometry><cylinder radius="0.045" length="0.08"/></geometry>
-        <material name="lidar_mount_gray"><color rgba="0.32 0.38 0.44 1"/></material>
-      </visual>
       <collision>
         <geometry><cylinder radius="0.08" length="0.11"/></geometry>
@@ -107,4 +92,17 @@
       <origin xyz="${xyz}" rpy="${rpy}"/>
     </joint>
+    <gazebo reference="${frame}"><material>Gazebo/Black</material></gazebo>
+    <xacro:fixed_cylinder_visual
+      name="${frame}_scan_band_link" parent="${frame}"
+      xyz="0 0 0" rpy="0 0 0" radius="0.084" length="0.045"
+      gazebo_material="Gazebo/Blue" rgba="0.03 0.35 0.68 1"/>
+    <xacro:fixed_cylinder_visual
+      name="${frame}_cap_link" parent="${frame}"
+      xyz="0 0 0.065" rpy="0 0 0" radius="0.065" length="0.025"
+      gazebo_material="Gazebo/Grey" rgba="0.32 0.38 0.44 1"/>
+    <xacro:fixed_cylinder_visual
+      name="${frame}_mount_link" parent="${frame}"
+      xyz="0 0 -0.095" rpy="0 0 0" radius="0.045" length="0.08"
+      gazebo_material="Gazebo/Grey" rgba="0.32 0.38 0.44 1"/>
     <gazebo reference="${frame}">
       <sensor name="mid360_lidar" type="ray">
@@ -147,17 +145,7 @@
                params="parent frame xyz rpy topic update_rate">
     <link name="${frame}">
-      <visual name="imu_body">
+      <visual>
         <geometry><box size="0.12 0.09 0.04"/></geometry>
         <material name="imu_black"><color rgba="0.025 0.03 0.035 1"/></material>
-      </visual>
-      <visual name="imu_top">
-        <origin xyz="0 0 0.023"/>
-        <geometry><box size="0.10 0.07 0.008"/></geometry>
-        <material name="imu_top_gray"><color rgba="0.32 0.38 0.44 1"/></material>
-      </visual>
-      <visual name="imu_forward_marker">
-        <origin xyz="0.045 0 0.031"/>
-        <geometry><box size="0.045 0.012 0.009"/></geometry>
-        <material name="imu_axis_red"><color rgba="0.90 0.05 0.05 1"/></material>
       </visual>
       <collision>
@@ -175,4 +163,13 @@
       <origin xyz="${xyz}" rpy="${rpy}"/>
     </joint>
+    <gazebo reference="${frame}"><material>Gazebo/Black</material></gazebo>
+    <xacro:fixed_box_visual
+      name="${frame}_top_link" parent="${frame}"
+      xyz="0 0 0.023" rpy="0 0 0" size="0.10 0.07 0.008"
+      gazebo_material="Gazebo/Grey" rgba="0.32 0.38 0.44 1"/>
+    <xacro:fixed_box_visual
+      name="${frame}_forward_marker_link" parent="${frame}"
+      xyz="0.045 0 0.031" rpy="0 0 0" size="0.045 0.012 0.009"
+      gazebo_material="Gazebo/Red" rgba="0.90 0.05 0.05 1"/>
     <gazebo reference="${frame}">
       <sensor name="imu_sensor" type="imu">
